File: pal-ntsc.kicad_sch (KiCad schematic)
At the start: 36 parts, among them U10 BT812, X2 30MHz

Commit message: update to kicad 9
Parts:
- C1, C10, C11, C12, C13, C14, C15, C16, C2, C3, C4, C47, C5, C6, C65, C66, C7, C8, C9, R12, R14, R19, R2, R20, R25, R27, R3, R35: footprint Resistor_SMD:R_1206_3216Metric_Pad1.24x1.80mm_HandSolder -> Resistor_SMD:R_1206_3216Metric_Pad1.30x1.75mm_HandSolder
- C62: footprint Resistor_SMD:R_1210_3225Metric_Pad1.24x2.70mm_HandSolder -> Resistor_SMD:R_1210_3225Metric_Pad1.30x2.65mm_HandSolder
- D1, D2, D3, D4: footprint Diode_THT:D_DO-34_SOD68_P7.62mm_Horizontal -> footprints:D_DO-34_SOD68_P7.62mm_Horizontal
- L4: footprint Resistor_SMD:R_1812_4532Metric_Pad1.24x3.50mm_HandSolder -> Resistor_SMD:R_1812_4532Metric_Pad1.30x3.40mm_HandSolder
